File: pcb/core_system/core_system.kicad_pcb (KiCad board)
At the start: 2 copper layers, 95 x 72 mm, 47 parts, among them J1 Battery, J10 Conn_01x02_Pin, J11 Conn_01x06_Pin, J12 Conn_01x03_Pin, J13 LED Segment, J6 Conn_01x06_Pin, J8 Conn_01x08_Pin, J9 Conn_01x06_Pin, Q1 2SC2712-Y, Q2 IRLML6344TRPBF, SW1 SW_SPDT, U1 MCP23017x-x-SP, U2 ESP32-DevKitC, U3 MT3608

Commit message: PCBのフィードバック対応
Parts:
- D1: value CUS01 -> 1N5819; footprint Diode_SMD:D_SOD-323_HandSoldering -> Diode_SMD:D_SOD-123
- J1: footprint Connector_JST:JST_PH_B2B-PH-K_1x02_P2.00mm_Vertical -> Connector_JST:JST_XH_B2B-XH-A_1x02_P2.50mm_Vertical
- moved J1 1.97 mm to (110.0, 36.7)
Connections:
- L1 pad 1: Net-(U3-EN) -> Net-(SW1-A)
- U3 pad 4: Net-(U3-EN) -> Net-(SW1-A)
Routing:
- net Net-(SW1-A): track 72.5 -> 79.7 mm
- net Net-(U3-EN): track 7.08 -> 0.00 mm
- net +BATT: track 11.7 -> 12.9 mm

Commit message: 基板フィードバック対応
Other:
- board text added: "v101"
- board text removed: "v100"
Changed lines of the file:
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@@
 		(tags "connector JST XH vertical")
 		(property "Reference" "J1"
-			(at 1.25 -3.55 270)
+			(at 4.4 4.8 0)
 			(layer "F.SilkS")
 			(effects
@@
 		(tags "connector JST XH vertical")
 		(property "Reference" "J8"
-			(at -3.9 0.6 0)
+			(at -2 4.9 0)
 			(layer "F.SilkS")
 			(effects
@@
 		(tags "capacitor electrolytic")
 		(property "Reference" "C1"
-			(at 2.4 -5.1 180)
+			(at 0.2 4.3 180)
 			(layer "F.SilkS")
 			(effects
@@
 		)
 		(property "Value" "100μ"
-			(at 0 4.35 180)
+			(at 3.1 4.5 180)
 			(layer "F.Fab")
 			(effects
@@
 		(tags "capacitor handsolder")
 		(property "Reference" "C2"
-			(at -0.2 -9 0)
+			(at -2.8 0 0)
 			(layer "F.SilkS")
 			(effects
@@
 		(layer "Edge.Cuts")
 	)
-	(gr_text "v100\n"
+	(gr_text "v101"
 		(at 42.2 90.1 0)
 		(layer "F.SilkS" knockout)
