File: pcb/core_system/core_system.kicad_sch (KiCad schematic)
At the start: 64 parts, among them J1 Battery, J10 Conn_01x02_Pin, J11 Conn_01x06_Pin, J12 Conn_01x03_Pin, J13 LED Segment, J6 Conn_01x06_Pin, J8 Conn_01x08_Pin, J9 Conn_01x06_Pin, Q1 2SC2712-Y, Q2 IRLML6344TRPBF, SW1 SW_SPDT, SW2 SW_Rotary_1x6_MP, SW3 RED, SW4 GREEN, SW5 YELLOW, SW6 BLUE, SW7 WHITE, U1 MCP23017x-x-SP, U2 ESP32-DevKitC, U3 MT3608

Commit message: PCBのフィードバック対応
Parts:
- D1: value CUS01 -> 1N5819; footprint Diode_SMD:D_SOD-323_HandSoldering -> Diode_SMD:D_SOD-123
- J1: footprint Connector_JST:JST_PH_B2B-PH-K_1x02_P2.00mm_Vertical -> Connector_JST:JST_XH_B2B-XH-A_1x02_P2.50mm_Vertical
Connections:
- net at L1.1, U3.4 (EN): now also C8.1, R3.2, SW1.1 (A), U3.5 (IN)
Changed lines of the file:
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@@
 	)
 	(junction
+		(at 97.79 29.21)
+		(diameter 0)
+		(color 0 0 0 0)
+	)
+	(junction
 		(at 201.93 147.32)
 		(diameter 0)
@@
 	(wire
 		(pts
+			(xy 97.79 29.21) (xy 99.06 29.21)
+		)
+		(stroke
+			(width 0)
+			(type default)
+		)
+	)
+	(wire
+		(pts
 			(xy 118.11 105.41) (xy 138.43 105.41)
 		)
@@
 	(wire
 		(pts
+			(xy 97.79 29.21) (xy 97.79 34.29)
+		)
+		(stroke
+			(width 0)
+			(type default)
+		)
+	)
+	(wire
+		(pts
 			(xy 82.55 223.52) (xy 85.09 223.52)
 		)
@@
 	(wire
 		(pts
-			(xy 97.79 19.05) (xy 97.79 34.29)
-		)
-		(stroke
-			(width 0)
-			(type default)
-		)
-	)
-	(wire
-		(pts
 			(xy 190.5 200.66) (xy 194.31 200.66)
 		)
@@
 	(wire
 		(pts
+			(xy 97.79 19.05) (xy 97.79 29.21)
+		)
+		(stroke
+			(width 0)
+			(type default)
+		)
+	)
+	(wire
+		(pts
 			(xy 359.41 143.51) (xy 369.57 143.51)
 		)
@@
 	(wire
 		(pts
-			(xy 93.98 29.21) (xy 99.06 29.21)
+			(xy 93.98 29.21) (xy 97.79 29.21)
 		)
 		(stroke
@@
 			)
 		)
-		(property "Footprint" "Connector_JST:JST_PH_B2B-PH-K_1x02_P2.00mm_Vertical"
+		(property "Footprint" "Connector_JST:JST_XH_B2B-XH-A_1x02_P2.50mm_Vertical"
 			(at 35.56 31.75 0)
 			(hide yes)
@@
 			)
 		)
-		(property "Value" "CUS01"
+		(property "Value" "1N5819"
 			(at 281.94 30.2261 90)
 			(show_name no)
@@
 			)
 		)
-		(property "Footprint" "Diode_SMD:D_SOD-323_HandSoldering"
+		(property "Footprint" "Diode_SMD:D_SOD-123"
 			(at 279.4 31.75 90)
 			(hide yes)

Commit message: 基板フィードバック対応
Parts:
- D4, SW4: value GREEN -> YELLOW
- D5, SW5: value YELLOW -> GREEN
Changed lines of the file:
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@@
 			)
 		)
-		(property "Value" "YELLOW"
+		(property "Value" "GREEN"
 			(at 260.35 186.69 0)
 			(show_name no)
@@
 			)
 		)
-		(property "Value" "GREEN"
+		(property "Value" "YELLOW"
 			(at 260.35 176.53 0)
 			(show_name no)
@@
 			)
 		)
-		(property "Value" "GREEN"
+		(property "Value" "YELLOW"
 			(at 319.9765 177.8 0)
 			(show_name no)
@@
 			)
 		)
-		(property "Value" "YELLOW"
+		(property "Value" "GREEN"
 			(at 319.9765 187.96 0)
 			(show_name no)
